File: PCB Dev/PCB_1_AK4619VN/PCB_1_AK4619VN.kicad_sch (KiCad schematic)
At the start: 7 parts

Commit message: yuh
Parts:
- removed C?: 0.1uF, symbol Device:C
- removed C?: 10uF, symbol Device:C_Polarized
- added C?: 10uF, symbol Device:C_Polarized
- added C?: 0.1uF, symbol Device:C
Connections:
- net AVDD is gone; now on net GND: U?.18 (AVDD)
- net GND: now also C?.1, C?.2
- net TVDD: now also C?.1, C?.2
