File: PCB Dev/PCB_1_AK4619VN/_autosave-PCB_1_AK4619VN.kicad_sch (KiCad schematic)
At the start: 13 parts

Commit message: lil pcb changes
Connections:
- net GND: now also P?.A1 (GND), P?.A12 (GND), P?.B1 (GND), P?.B12 (GND), P?.S1 (SHIELD)
Changed lines of the file:
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@@
+    (stroke (width 0) (type default) (color 0 0 0 0))
+  )
+  (wire (pts (xy 68.58 185.42) (xy 81.28 185.42))
     (stroke (width 0) (type default) (color 0 0 0 0))
   )
@@
     (stroke (width 0) (type default) (color 0 0 0 0))
   )
+  (wire (pts (xy 68.58 190.5) (xy 81.28 190.5))
+    (stroke (width 0) (type default) (color 0 0 0 0))
+  )
   (wire (pts (xy 189.23 58.42) (xy 181.61 58.42))
     (stroke (width 0) (type default) (color 0 0 0 0))
@@
   )
   (wire (pts (xy 285.75 93.98) (xy 285.75 100.33))
+    (stroke (width 0) (type default) (color 0 0 0 0))
+  )
+  (wire (pts (xy 68.58 172.72) (xy 81.28 172.72))
     (stroke (width 0) (type default) (color 0 0 0 0))
   )
@@
     )
     (property "Datasheet" "" (id 3) (at 176.53 73.66 0)
+      (effects (font (size 1.27 1.27)) hide)
+    )
+    (pin "1")
+  )
+  (symbol (lib_id "power:GND") (at 45.72 210.82 0) (unit 1)
+    (in_bom yes) (on_board yes) (fields_autoplaced)
+    (property "Reference" "#PWR?" (id 0) (at 45.72 217.17 0)
+      (effects (font (size 1.27 1.27)) hide)
+    )
+    (property "Value" "GND" (id 1) (at 45.72 215.9 0))
+    (property "Footprint" "" (id 2) (at 45.72 210.82 0)
+      (effects (font (size 1.27 1.27)) hide)
+    )
+    (property "Datasheet" "" (id 3) (at 45.72 210.82 0)
       (effects (font (size 1.27 1.27)) hide)
     )
@@
     (pin "2")
   )
+  (symbol (lib_id "power:GND") (at 53.34 210.82 0) (unit 1)
+    (in_bom yes) (on_board yes) (fields_autoplaced)
+    (property "Reference" "#PWR?" (id 0) (at 53.34 217.17 0)
+      (effects (font (size 1.27 1.27)) hide)
+    )
+    (property "Value" "GND" (id 1) (at 53.34 215.9 0))
+    (property "Footprint" "" (id 2) (at 53.34 210.82 0)
+      (effects (font (size 1.27 1.27)) hide)
+    )
+    (property "Datasheet" "" (id 3) (at 53.34 210.82 0)
+      (effects (font (size 1.27 1.27)) hide)
+    )
+    (pin "1")
+  )
   (symbol (lib_id "power:GND") (at 273.05 104.14 0) (unit 1)
     (in_bom yes) (on_board yes)
@@
       (reference "#PWR?") (unit 1) (value "GND") (footprint "")
     )
+    (path "/3cc00b7e-59e2-49fb-82da-4416ce5fd88d"
+      (reference "#PWR?") (unit 1) (value "GND") (footprint "")
+    )
     (path "/466f8cae-d802-4736-82c3-9d61958ec3ab"
       (reference "#PWR?") (unit 1) (value "GND") (footprint "")
     )
+    (path "/7d1e7eed-b098-448f-ad02-474c81ceb908"
+      (reference "#PWR?") (unit 1) (value "GND") (footprint "")
+    )
