File: PCB Dev/Player V1/_autosave-PlayerV1.kicad_sch (KiCad schematic)
At the start: 54 parts, among them J1 USB_C_Receptacle_USB2.0, J2 Conn_01x02_Female, J3 Conn_01x02_Female, J4 Conn_01x02_Female, J5 SJ-43516-SMT-U, J6 SJ-43516-SMT-U, U1 AP7217A, U2 AK4619VN, U3 TP4056, U4 ESP32-S3-WROOM-1-N8

Commit message: PCB Dev
Added headphone jacks amp, and stereo speakers amp

added gui interface buttons though they may have to be put in another pcb

learned esp32 s3 does not have bluetooth a2dp so I need to switch to esp32 wroom 32E with 16mb instead only issue is gpio are becoming scarce
Parts:
- added C3, C5: 1uF, Capacitor_SMD:C_0805_2012Metric, symbol Device:C
- added R6: 100K, symbol Device:R
- added U3: AP7217A, AP7217A:SOIC127P600X175-8N, symbol AP7217A:AP7217A
- renumbered C10 to C1, C5 to C10, C6 to C11, C7 to C12, C8 to C13, C20 to C16, C21 to C17, C22 to C18, C23 to C19, C1 to C2, C9 to C20, C13 to C21, C24 to C22, C25 to C23, C16 to C24, C17 to C25, C18 to C26, C19 to C27, C26 to C28, C27 to C29, C2 to C4, C11 to C6, C3 to C7, C12 to C8, C4 to C9, EVP-BT7A4A0 to EVP-BT7A4A1, EVP-BT7A4A1 to EVP-BT7A4A2, EVP-BT7A4A2 to EVP-BT7A4A3, EVP-BT7A4A3 to EVP-BT7A4A4, J5 to J3, J6 to J4, J3 to J5, J4 to J6, R2 to R1, R3 to R2, R4 to R3, R5 to R4, R1 to R5, R6 to R7, U3 to U1, U1 to U2, U2 to U5
Connections:
- net +BATT: now also C5.2, R6.2, U3.4 (Vin), U3.8 (EN)
- net GND: now also C3.1, C5.1, U3.1 (GND), U3.3 (GND), U3.5 (GND), U3.7 (GND)
- new net: R6.1, U3.6 (VDo)
- new net VDC: C3.2, U3.2 (VRo)
