File: PCB Dev/Player V1/PlayerV1.1_MotherBoard/PlayerV1.1_MotherBoard.kicad_sch (KiCad schematic)
At the start: 73 parts, among them J1 USB_C_Receptacle_USB2.0, J2 Conn_01x02_Female, J3 SJ-3524-SMT-BE, Q1 Q_NPN_BEC, Q2 Q_NPN_BEC, U1 MIC5213-2.5YC5-TR, U2 TP4056, U3 AP7217A, U4 CP2102N-A02-GQFN28R, U5 BQ27441DRZR-G1A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

Commit message: quick update
:)
Parts:
- gave numbers to parts that had none: 4
- renumbered 11 to 111, C9 to C10, C10 to C11, C13 to C12, C11 to C13, C17 to C19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
