File: PCB Dev/Player V1/PlayerV1.1_MotherBoard/PlayerV1.1_MotherBoard.kicad_sch (KiCad schematic)
At the start: 74 parts, among them J1 USB_C_Receptacle_USB2.0, J2 Conn_01x02_Female, J4 SJ-3524-SMT-BE, Q1 Q_NPN_BEC, Q2 Q_NPN_BEC, U1 MIC5213-2.5YC5-TR, U2 TP4056, U3 AP7217A, U4 CP2102N-A02-GQFN28R, U5 BQ27441DRZR-G1A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

Commit message: code
had to revise the code for the display and the audio so both can operate at the same time

using dma on both aspects already
dma on the display fixed it's operation issues
though dma was already in use on the i2s port and it was still stuttering so I have almost no official idea what the issue actually is
though, apparently the i2s amp i am currently using may be the issue so well have to make the official prototype then see
because then i wont have to worry about
Parts:
- removed J2, SPK1, SPK2: Conn_01x02_Female, symbol Connector:Conn_01x02_Female
- added J2: B2B-PH-SM4-TBLFSN, CONN_B2B-PH-SM4-TBLFSN_JST, symbol JST_B2B-PH-SM4-TB:B2B-PH-SM4-TBLFSN
- added J5: SPK1, CONN_B2B-PH-SM4-TBLFSN_JST, symbol JST_B2B-PH-SM4-TB:B2B-PH-SM4-TBLFSN
- added J6: SPK2, CONN_B2B-PH-SM4-TBLFSN_JST, symbol JST_B2B-PH-SM4-TB:B2B-PH-SM4-TBLFSN
- D1, D2: footprint (none) -> LED_SMD:LED_0201_0603Metric_Pad0.64x0.40mm_HandSolder
- gave numbers to parts that had none: 1
Connections:
- net +BATT: now also J2.2
- net GND: now also GUI_In/Output1.11, J2.1
- net VCC: now also GUI_In/Output1.12
- net VCLK: now also Cell_Input1.5; no longer Cell_Input1.4
- net VCS: now also Cell_Input1.6; no longer Cell_Input1.3
- net VMISO: now also Cell_Input1.4; no longer Cell_Input1.6
- net VMOSI: now also Cell_Input1.3; no longer Cell_Input1.5
- net at j3.22 (RLS-): now also J5.1
- net at j3.23 (RLS+): now also J5.2
- net at j3.19 (LLS+): now also J6.2
- net at j3.20 (LLS-): now also J6.1

Commit message: yuh
Parts:
- added U?: AK4619VN, AK4619VN_AKM, symbol AK4619VN:AK4619VN
Changed lines of the file:
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@@
     (pin "2")
+  )
+  (symbol (lib_id "AK4619VN:AK4619VN") (at 325.12 120.65 0) (unit 1)
+    (in_bom yes) (on_board yes) (fields_autoplaced)
+    (property "Reference" "U?" (id 0) (at 363.22 109.22 0)
+      (effects (font (size 1.524 1.524)))
+    )
+    (property "Value" "AK4619VN" (id 1) (at 363.22 113.03 0)
+      (effects (font (size 1.524 1.524)))
+    )
+    (property "Footprint" "AK4619VN_AKM" (id 2) (at 325.12 120.65 0)
+      (effects (font (size 1.27 1.27) italic) hide)
+    )
+    (property "Datasheet" "AK4619VN" (id 3) (at 325.12 120.65 0)
+      (effects (font (size 1.27 1.27) italic) hide)
+    )
+    (pin "1")
+    (pin "10")
+    (pin "11")
+    (pin "12")
+    (pin "13")
+    (pin "14")
+    (pin "15")
+    (pin "16")
+    (pin "17")
+    (pin "18")
+    (pin "19")
+    (pin "2")
+    (pin "20")
+    (pin "21")
+    (pin "22")
+    (pin "23")
+    (pin "24")
+    (pin "25")
+    (pin "26")
+    (pin "27")
+    (pin "28")
+    (pin "29")
+    (pin "3")
+    (pin "30")
+    (pin "31")
+    (pin "32")
+    (pin "33")
+    (pin "4")
+    (pin "5")
+    (pin "6")
+    (pin "7")
+    (pin "8")
+    (pin "9")
   )
   (symbol (lib_id "power:GND") (at 403.86 77.47 270) (unit 1)
@@
       (reference "U7") (unit 1) (value "MCP23017-E/ML") (footprint "MCP23017_E_ML:QFN28_6x6MC_MCH")
     )
+    (path "/cd818bb9-b05a-40d3-88b4-1d88083d1122"
+      (reference "U?") (unit 1) (value "AK4619VN") (footprint "AK4619VN_AKM")
+    )
     (path "/85e2d2ff-9e64-4772-8d49-2f864f93431c"
