File: PCB Dev/Player V1/PlayerV1.1_MotherBoard/_autosave-PlayerV1.1_MotherBoard.kicad_sch (KiCad schematic)
At the start: 74 parts, among them J1 USB_C_Receptacle_USB2.0, J2 Conn_01x02_Female, J4 SJ-3524-SMT-BE, Q1 Q_NPN_BEC, Q2 Q_NPN_BEC, U1 MIC5213-2.5YC5-TR, U2 TP4056, U3 AP7217A, U4 CP2102N-A02-GQFN28R, U5 BQ27441DRZR-G1A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

Commit message: added all jst connectors
new upward facing jst connectors
fixed footprint issue on the usbC port that resulted in a malformed board outline
need to add holes for the usbc port somehow
need to start laying out the pcb after using the component measurements to make proper pcb heights, cutouts, and tactile buttons
Parts:
- removed J2, SPK1, SPK2: Conn_01x02_Female, symbol Connector:Conn_01x02_Female
- added J?: SPK2, CONN_B2B-PH-SM4-TBLFSN_JST, symbol JST_B2B-PH-SM4-TB:B2B-PH-SM4-TBLFSN
- added J?: B2B-PH-SM4-TBLFSN, CONN_B2B-PH-SM4-TBLFSN_JST, symbol JST_B2B-PH-SM4-TB:B2B-PH-SM4-TBLFSN
- added J?: SPK1, CONN_B2B-PH-SM4-TBLFSN_JST, symbol JST_B2B-PH-SM4-TB:B2B-PH-SM4-TBLFSN
- D1, D2: footprint (none) -> LED_SMD:LED_0201_0603Metric_Pad0.64x0.40mm_HandSolder
- gave numbers to parts that had none: 1
Connections:
- net +BATT: now also J?.2
- net GND: now also GUI_In/Output1.11, J?.1
- net VCC: now also GUI_In/Output1.12
- net at j3.22 (RLS-): now also J?.1
- net at j3.23 (RLS+): now also J?.2
- net at j3.19 (LLS+): now also J?.2
- net at j3.20 (LLS-): now also J?.1
